File: pcbs/BinaryClock.sch (KiCad schematic (older format))
At the start: 33 parts, among them IC1 ATTINY2313A-S, P1 USB_OTG, P2 CONN_02X03, SW1 SW_PUSH, U1 FT230XS, U2 STP16CPC26, U3 DS3231M

Commit message: Fixed routing issues, fixed paste layer issues, and eliminated electrolytic caps
Parts:
- removed 2K1: POT, TylerCustom:pot_trimmer_smd, symbol POT
- removed C2, C7: 10 uF, Capacitors_SMD:c_elec_6.3x5.7, symbol CP
- removed R1: 1K8, Resistors_SMD:R_0805, symbol R
- added C1: .1 uF, Capacitors_SMD:C_0805, symbol C_Small
- added C10: 0.1 uF, Resistors_SMD:R_0805, symbol C
- added C2: 47 pF, symbol C_Small
- added C3: 47 pF, Capacitors_SMD:C_0805, symbol C_Small
- added C5: 4.7 uF, Resistors_SMD:R_0805, symbol C
- added R6: 2K, Resistors_SMD:R_0805, symbol R
- added W11, W12, W13, W14: TEST_1P, Measurement_Points:Measurement_Point_Round-SMD-Pad_Small, symbol TEST_1P
- W1, W2: footprint Measurement_Points:Measurement_Point_Round-SMD-Pad_Small -> Measurement_Points:Measurement_Point_Square-SMD-Pad_Big
- W10, W9: footprint Measurement_Points:Test_Point_Keystone_5019_Minature -> Measurement_Points:Measurement_Point_Round-SMD-Pad_Small
- W3, W4: footprint Measurement_Points:Test_Point_Keystone_5019_Minature -> Measurement_Points:Measurement_Point_Square-SMD-Pad_Big
- renumbered C1 to C4, C3 to C6, C4 to C7, C5 to C8, C6 to C9
Connections:
- net +5V: now also C5.1
- net +BATT: now also C10.1
- net GND: now also C1.2, C10.2, C2.2, C3.2, C5.2, R6.2
- net RTC_SCL: now also W9.1
- net RTC_SDA: now also W10.1
- net UART_RXD: now also U1.1 (TXD), W11.1; no longer U1.4 (RXD)
- net UART_TXD: now also U1.4 (RXD), W12.1; no longer U1.1 (TXD)
- net ~RST: no longer U1.11 (~RESET)
- net at U2.23 (R-EXT): now also R6.1
- net at U1.10 (3V3OUT), U1.3 (VCCIO): now also U1.11 (~RESET), C1.1
- net at P1.2 (D-), R3.1: now also C2.1
- net at P1.3 (D+), R4.1: now also C3.1
- net at IC1.5 (PA0(XTAL1/CLKI/PCINT8)): now also W13.1
- net at IC1.6 ((PCINT13/CKOUT/XCK/INT0)PD2): now also W14.1
- no-connect marks 17 -> 14
Other:
- moved on the sheet: C4, P1, W1, W2
